Commit message: add test

File: assets/urdf/ycb/011_banana/011_banana.urdf (robot description, URDF)
Before this commit: robot banana, 1 links, 0 joints
Links:
- link banana: geometry collision mesh filename=./collision.obj scale=0.01 0.01 0.01; visual mesh filename=./textured.obj scale=0.01 0.01 0.01
