Commit message: 2024.04.15 加了麦轮但是注释掉了

File: assets/urdf/robomasterEP_description/robot/robomaster.urdf (robot description, URDF)
Before this commit: robot robomaster_ep, 39 links, 38 joints
Links:
- link front_left_wheel_link: geometry collision mesh filename=../meshes/mecanum_wheel.stl scale=0.6 0.6 0.6; visual cylinder length=0.001 radius=0.007
- link front_right_wheel_link: geometry collision mesh filename=../meshes/mecanum_wheel.stl scale=0.6 0.6 0.6; visual cylinder length=0.001 radius=0.007
- link rear_left_wheel_link: geometry collision mesh filename=../meshes/mecanum_wheel.stl scale=0.6 0.6 0.6; visual cylinder length=0.001 radius=0.007
- link rear_right_wheel_link: geometry collision mesh filename=../meshes/mecanum_wheel.stl scale=0.6 0.6 0.6; visual cylinder length=0.001 radius=0.007
