Commit message: 2024.04.16 添加了麦轮，可以正常转弯等

File: assets/urdf/robomasterEP_description/robot/robomaster.urdf (robot description, URDF)
Before this commit: robot robomaster_ep, 39 links, 38 joints
Links:
- added link front_left_roller10_link, mass 0.3; collision mesh filename=../meshes/mecanum_roller.stl scale=0.6 0.6 0.6; visual mesh filename=../meshes/mecanum_roller.dae scale=0.6 0.6 0.6
- added link front_left_roller11_link, mass 0.3; collision mesh filename=../meshes/mecanum_roller.stl scale=0.6 0.6 0.6; visual mesh filename=../meshes/mecanum_roller.dae scale=0.6 0.6 0.6
- added link front_left_roller12_link, mass 0.3; collision mesh filename=../meshes/mecanum_roller.stl scale=0.6 0.6 0.6; visual mesh filename=../meshes/mecanum_roller.dae scale=0.6 0.6 0.6
- added link front_left_roller13_link, mass 0.3; collision mesh filename=../meshes/mecanum_roller.stl scale=0.6 0.6 0.6; visual mesh filename=../meshes/mecanum_roller.dae scale=0.6 0.6 0.6
- added link front_left_roller14_link, mass 0.3; collision mesh filename=../meshes/mecanum_roller.stl scale=0.6 0.6 0.6; visual mesh filename=../meshes/mecanum_roller.dae scale=0.6 0.6 0.6
- added link front_left_roller15_link, mass 0.3; collision mesh filename=../meshes/mecanum_roller.stl scale=0.6 0.6 0.6; visual mesh filename=../meshes/mecanum_roller.dae scale=0.6 0.6 0.6
- added link front_left_roller1_link, mass 0.3; collision mesh filename=../meshes/mecanum_roller.stl scale=0.6 0.6 0.6; visual mesh filename=../meshes/mecanum_roller.dae scale=0.6 0.6 0.6
- added link front_left_roller2_link, mass 0.3; collision mesh filename=../meshes/mecanum_roller.stl scale=0.6 0.6 0.6; visual mesh filename=../meshes/mecanum_roller.dae scale=0.6 0.6 0.6
- added link front_left_roller3_link, mass 0.3; collision mesh filename=../meshes/mecanum_roller.stl scale=0.6 0.6 0.6; visual mesh filename=../meshes/mecanum_roller.dae scale=0.6 0.6 0.6
- added link front_left_roller4_link, mass 0.3; collision mesh filename=../meshes/mecanum_roller.stl scale=0.6 0.6 0.6; visual mesh filename=../meshes/mecanum_roller.dae scale=0.6 0.6 0.6
- added link front_left_roller5_link, mass 0.3; collision mesh filename=../meshes/mecanum_roller.stl scale=0.6 0.6 0.6; visual mesh filename=../meshes/mecanum_roller.dae scale=0.6 0.6 0.6
- added link front_left_roller6_link, mass 0.3; collision mesh filename=../meshes/mecanum_roller.stl scale=0.6 0.6 0.6; visual mesh filename=../meshes/mecanum_roller.dae scale=0.6 0.6 0.6
- added link front_left_roller7_link, mass 0.3; collision mesh filename=../meshes/mecanum_roller.stl scale=0.6 0.6 0.6; visual mesh filename=../meshes/mecanum_roller.dae scale=0.6 0.6 0.6
- added link front_left_roller8_link, mass 0.3; collision mesh filename=../meshes/mecanum_roller.stl scale=0.6 0.6 0.6; visual mesh filename=../meshes/mecanum_roller.dae scale=0.6 0.6 0.6
- added link front_left_roller9_link, mass 0.3; collision mesh filename=../meshes/mecanum_roller.stl scale=0.6 0.6 0.6; visual mesh filename=../meshes/mecanum_roller.dae scale=0.6 0.6 0.6
- added link front_right_roller10_link, mass 0.3; collision mesh filename=../meshes/mecanum_roller.stl scale=0.6 0.6 0.6; visual mesh filename=../meshes/mecanum_roller.dae scale=0.6 0.6 0.6
- added link front_right_roller11_link, mass 0.3; collision mesh filename=../meshes/mecanum_roller.stl scale=0.6 0.6 0.6; visual mesh filename=../meshes/mecanum_roller.dae scale=0.6 0.6 0.6
- added link front_right_roller12_link, mass 0.3; collision mesh filename=../meshes/mecanum_roller.stl scale=0.6 0.6 0.6; visual mesh filename=../meshes/mecanum_roller.dae scale=0.6 0.6 0.6
- added link front_right_roller13_link, mass 0.3; collision mesh filename=../meshes/mecanum_roller.stl scale=0.6 0.6 0.6; visual mesh filename=../meshes/mecanum_roller.dae scale=0.6 0.6 0.6
- added link front_right_roller14_link, mass 0.3; collision mesh filename=../meshes/mecanum_roller.stl scale=0.6 0.6 0.6; visual mesh filename=../meshes/mecanum_roller.dae scale=0.6 0.6 0.6
- added link front_right_roller15_link, mass 0.3; collision mesh filename=../meshes/mecanum_roller.stl scale=0.6 0.6 0.6; visual mesh filename=../meshes/mecanum_roller.dae scale=0.6 0.6 0.6
- added link front_right_roller1_link, mass 0.3; collision mesh filename=../meshes/mecanum_roller.stl scale=0.6 0.6 0.6; visual mesh filename=../meshes/mecanum_roller.dae scale=0.6 0.6 0.6
- added link front_right_roller2_link, mass 0.3; collision mesh filename=../meshes/mecanum_roller.stl scale=0.6 0.6 0.6; visual mesh filename=../meshes/mecanum_roller.dae scale=0.6 0.6 0.6
- added link front_right_roller3_link, mass 0.3; collision mesh filename=../meshes/mecanum_roller.stl scale=0.6 0.6 0.6; visual mesh filename=../meshes/mecanum_roller.dae scale=0.6 0.6 0.6
- added link front_right_roller4_link, mass 0.3; collision mesh filename=../meshes/mecanum_roller.stl scale=0.6 0.6 0.6; visual mesh filename=../meshes/mecanum_roller.dae scale=0.6 0.6 0.6
- added link front_right_roller5_link, mass 0.3; collision mesh filename=../meshes/mecanum_roller.stl scale=0.6 0.6 0.6; visual mesh filename=../meshes/mecanum_roller.dae scale=0.6 0.6 0.6
- added link front_right_roller6_link, mass 0.3; collision mesh filename=../meshes/mecanum_roller.stl scale=0.6 0.6 0.6; visual mesh filename=../meshes/mecanum_roller.dae scale=0.6 0.6 0.6
- added link front_right_roller7_link, mass 0.3; collision mesh filename=../meshes/mecanum_roller.stl scale=0.6 0.6 0.6; visual mesh filename=../meshes/mecanum_roller.dae scale=0.6 0.6 0.6
- added link front_right_roller8_link, mass 0.3; collision mesh filename=../meshes/mecanum_roller.stl scale=0.6 0.6 0.6; visual mesh filename=../meshes/mecanum_roller.dae scale=0.6 0.6 0.6
- added link front_right_roller9_link, mass 0.3; collision mesh filename=../meshes/mecanum_roller.stl scale=0.6 0.6 0.6; visual mesh filename=../meshes/mecanum_roller.dae scale=0.6 0.6 0.6
- added link rear_left_roller10_link, mass 0.3; collision mesh filename=../meshes/mecanum_roller.stl scale=0.6 0.6 0.6; visual mesh filename=../meshes/mecanum_roller.dae scale=0.6 0.6 0.6
- added link rear_left_roller11_link, mass 0.3; collision mesh filename=../meshes/mecanum_roller.stl scale=0.6 0.6 0.6; visual mesh filename=../meshes/mecanum_roller.dae scale=0.6 0.6 0.6
- added link rear_left_roller12_link, mass 0.3; collision mesh filename=../meshes/mecanum_roller.stl scale=0.6 0.6 0.6; visual mesh filename=../meshes/mecanum_roller.dae scale=0.6 0.6 0.6
- added link rear_left_roller13_link, mass 0.3; collision mesh filename=../meshes/mecanum_roller.stl scale=0.6 0.6 0.6; visual mesh filename=../meshes/mecanum_roller.dae scale=0.6 0.6 0.6
- added link rear_left_roller14_link, mass 0.3; collision mesh filename=../meshes/mecanum_roller.stl scale=0.6 0.6 0.6; visual mesh filename=../meshes/mecanum_roller.dae scale=0.6 0.6 0.6
- added link rear_left_roller15_link, mass 0.3; collision mesh filename=../meshes/mecanum_roller.stl scale=0.6 0.6 0.6; visual mesh filename=../meshes/mecanum_roller.dae scale=0.6 0.6 0.6
- added link rear_left_roller1_link, mass 0.3; collision mesh filename=../meshes/mecanum_roller.stl scale=0.6 0.6 0.6; visual mesh filename=../meshes/mecanum_roller.dae scale=0.6 0.6 0.6
- added link rear_left_roller2_link, mass 0.3; collision mesh filename=../meshes/mecanum_roller.stl scale=0.6 0.6 0.6; visual mesh filename=../meshes/mecanum_roller.dae scale=0.6 0.6 0.6
- added link rear_left_roller3_link, mass 0.3; collision mesh filename=../meshes/mecanum_roller.stl scale=0.6 0.6 0.6; visual mesh filename=../meshes/mecanum_roller.dae scale=0.6 0.6 0.6
- added link rear_left_roller4_link, mass 0.3; collision mesh filename=../meshes/mecanum_roller.stl scale=0.6 0.6 0.6; visual mesh filename=../meshes/mecanum_roller.dae scale=0.6 0.6 0.6
- added link rear_left_roller5_link, mass 0.3; collision mesh filename=../meshes/mecanum_roller.stl scale=0.6 0.6 0.6; visual mesh filename=../meshes/mecanum_roller.dae scale=0.6 0.6 0.6
- added link rear_left_roller6_link, mass 0.3; collision mesh filename=../meshes/mecanum_roller.stl scale=0.6 0.6 0.6; visual mesh filename=../meshes/mecanum_roller.dae scale=0.6 0.6 0.6
- added link rear_left_roller7_link, mass 0.3; collision mesh filename=../meshes/mecanum_roller.stl scale=0.6 0.6 0.6; visual mesh filename=../meshes/mecanum_roller.dae scale=0.6 0.6 0.6
- added link rear_left_roller8_link, mass 0.3; collision mesh filename=../meshes/mecanum_roller.stl scale=0.6 0.6 0.6; visual mesh filename=../meshes/mecanum_roller.dae scale=0.6 0.6 0.6
- added link rear_left_roller9_link, mass 0.3; collision mesh filename=../meshes/mecanum_roller.stl scale=0.6 0.6 0.6; visual mesh filename=../meshes/mecanum_roller.dae scale=0.6 0.6 0.6
- added link rear_right_roller10_link, mass 0.3; collision mesh filename=../meshes/mecanum_roller.stl scale=0.6 0.6 0.6; visual mesh filename=../meshes/mecanum_roller.dae scale=0.6 0.6 0.6
- added link rear_right_roller11_link, mass 0.3; collision mesh filename=../meshes/mecanum_roller.stl scale=0.6 0.6 0.6; visual mesh filename=../meshes/mecanum_roller.dae scale=0.6 0.6 0.6
- added link rear_right_roller12_link, mass 0.3; collision mesh filename=../meshes/mecanum_roller.stl scale=0.6 0.6 0.6; visual mesh filename=../meshes/mecanum_roller.dae scale=0.6 0.6 0.6
- added link rear_right_roller13_link, mass 0.3; collision mesh filename=../meshes/mecanum_roller.stl scale=0.6 0.6 0.6; visual mesh filename=../meshes/mecanum_roller.dae scale=0.6 0.6 0.6
- added link rear_right_roller14_link, mass 0.3; collision mesh filename=../meshes/mecanum_roller.stl scale=0.6 0.6 0.6; visual mesh filename=../meshes/mecanum_roller.dae scale=0.6 0.6 0.6
- added link rear_right_roller15_link, mass 0.3; collision mesh filename=../meshes/mecanum_roller.stl scale=0.6 0.6 0.6; visual mesh filename=../meshes/mecanum_roller.dae scale=0.6 0.6 0.6
- added link rear_right_roller1_link, mass 0.3; collision mesh filename=../meshes/mecanum_roller.stl scale=0.6 0.6 0.6; visual mesh filename=../meshes/mecanum_roller.dae scale=0.6 0.6 0.6
- added link rear_right_roller2_link, mass 0.3; collision mesh filename=../meshes/mecanum_roller.stl scale=0.6 0.6 0.6; visual mesh filename=../meshes/mecanum_roller.dae scale=0.6 0.6 0.6
- added link rear_right_roller3_link, mass 0.3; collision mesh filename=../meshes/mecanum_roller.stl scale=0.6 0.6 0.6; visual mesh filename=../meshes/mecanum_roller.dae scale=0.6 0.6 0.6
- added link rear_right_roller4_link, mass 0.3; collision mesh filename=../meshes/mecanum_roller.stl scale=0.6 0.6 0.6; visual mesh filename=../meshes/mecanum_roller.dae scale=0.6 0.6 0.6
- added link rear_right_roller5_link, mass 0.3; collision mesh filename=../meshes/mecanum_roller.stl scale=0.6 0.6 0.6; visual mesh filename=../meshes/mecanum_roller.dae scale=0.6 0.6 0.6
- added link rear_right_roller6_link, mass 0.3; collision mesh filename=../meshes/mecanum_roller.stl scale=0.6 0.6 0.6; visual mesh filename=../meshes/mecanum_roller.dae scale=0.6 0.6 0.6
- added link rear_right_roller7_link, mass 0.3; collision mesh filename=../meshes/mecanum_roller.stl scale=0.6 0.6 0.6; visual mesh filename=../meshes/mecanum_roller.dae scale=0.6 0.6 0.6
- added link rear_right_roller8_link, mass 0.3; collision mesh filename=../meshes/mecanum_roller.stl scale=0.6 0.6 0.6; visual mesh filename=../meshes/mecanum_roller.dae scale=0.6 0.6 0.6
- added link rear_right_roller9_link, mass 0.3; collision mesh filename=../meshes/mecanum_roller.stl scale=0.6 0.6 0.6; visual mesh filename=../meshes/mecanum_roller.dae scale=0.6 0.6 0.6
- link front_left_wheel_link: mass 0.162 -> 2.0; geometry collision mesh filename=../meshes/mecanum_wheel.stl scale=0.6 0.6 0.6; visual mesh filename=../meshes/mecanum_wheel.dae scale=0.6 0.6 0.6
- link front_right_wheel_link: mass 0.162 -> 2.0; geometry collision mesh filename=../meshes/mecanum_wheel.stl scale=0.6 0.6 0.6; visual mesh filename=../meshes/mecanum_wheel.dae scale=0.6 0.6 0.6
- link rear_left_wheel_link: mass 0.162 -> 2.0; geometry collision mesh filename=../meshes/mecanum_wheel.stl scale=0.6 0.6 0.6; visual mesh filename=../meshes/mecanum_wheel.dae scale=0.6 0.6 0.6
- link rear_right_wheel_link: mass 0.162 -> 2.0; geometry collision mesh filename=../meshes/mecanum_wheel.stl scale=0.6 0.6 0.6; visual mesh filename=../meshes/mecanum_wheel.dae scale=0.6 0.6 0.6
Joints:
- added joint front_left_roller10_joint: type continuous, parent front_left_wheel_link, child front_left_roller10_link, origin xyz=0 -0.04344421259793468 -0.0315640680481058 rpy=-0.7989541677433551 0.6090169187607924 0.5313896516603533, axis 1 0 0
- added joint front_left_roller11_joint: type continuous, parent front_left_wheel_link, child front_left_roller11_link, origin xyz=0 -0.026850000000000023 -0.04650556418322434 rpy=-1.1831996401397156 0.3613671239067081 0.7137243789447655, axis 1 0 0
- added joint front_left_roller12_joint: type continuous, parent front_left_wheel_link, child front_left_roller12_link, origin xyz=0 -0.0056131784774729855 -0.05340582578127628 rpy=-1.4966127917301506 0.07398025001120935 0.7826515949744619, axis 1 0 0
- added joint front_left_roller13_joint: type continuous, parent front_left_wheel_link, child front_left_roller13_link, origin xyz=0 0.01659421259793466 -0.051071734925049746 rpy=1.3449626171032882 -0.22028527385474703 0.7603177925108144, axis 1 0 0
- added joint front_left_roller14_joint: type continuous, parent front_left_wheel_link, child front_left_roller14_link, origin xyz=0 0.03593231356147066 -0.039906877128136085 rpy=1.0038406803226874 -0.4928592704898482 0.6390993414905143, axis 1 0 0
- added joint front_left_roller15_joint: type continuous, parent front_left_wheel_link, child front_left_roller15_link, origin xyz=0 0.04905739107540767 -0.021841757733170465 rpy=0.5619350361043127 -0.7022987807291682 0.38630030387691144, axis 1 0 0
- added joint front_left_roller1_joint: type continuous, parent front_left_wheel_link, child front_left_roller1_link, origin xyz=0 0.0537 0.0 rpy=-0.0 -0.7853981633974482 -0.0, axis 1 0 0
- added joint front_left_roller2_joint: type continuous, parent front_left_wheel_link, child front_left_roller2_link, origin xyz=0 0.049057391075407665 0.02184175773317047 rpy=-0.5619350361043128 -0.702298780729168 -0.3863003038769115, axis 1 0 0
- added joint front_left_roller3_joint: type continuous, parent front_left_wheel_link, child front_left_roller3_link, origin xyz=0 0.03593231356147068 0.03990687712813607 rpy=-1.0038406803226867 -0.4928592704898485 -0.6390993414905141, axis 1 0 0
- added joint front_left_roller4_joint: type continuous, parent front_left_wheel_link, child front_left_roller4_link, origin xyz=0 0.016594212597934678 0.051071734925049746 rpy=-1.3449626171032882 -0.2202852738547472 -0.7603177925108144, axis 1 0 0
- added joint front_left_roller5_joint: type continuous, parent front_left_wheel_link, child front_left_roller5_link, origin xyz=0 -0.005613178477472996 0.05340582578127627 rpy=1.4966127917301504 0.07398025001120949 -0.7826515949744619, axis 1 0 0
- added joint front_left_roller6_joint: type continuous, parent front_left_wheel_link, child front_left_roller6_link, origin xyz=0 -0.026849999999999985 0.04650556418322435 rpy=1.1831996401397162 0.3613671239067076 -0.7137243789447657, axis 1 0 0
- added joint front_left_roller7_joint: type continuous, parent front_left_wheel_link, child front_left_roller7_link, origin xyz=0 -0.04344421259793467 0.03156406804810581 rpy=0.7989541677433554 0.6090169187607923 -0.5313896516603536, axis 1 0 0
- added joint front_left_roller8_joint: type continuous, parent front_left_wheel_link, child front_left_roller8_link, origin xyz=0 -0.05252652615940536 0.011164857796913676 rpy=0.2920075036845471 0.7637777909460687 -0.20499125187874387, axis 1 0 0
- added joint front_left_roller9_joint: type continuous, parent front_left_wheel_link, child front_left_roller9_link, origin xyz=0 -0.052526526159405354 -0.011164857796913686 rpy=-0.29200750368454736 0.7637777909460687 0.20499125187874406, axis 1 0 0
- added joint front_right_roller10_joint: type continuous, parent front_right_wheel_link, child front_right_roller10_link, origin xyz=0 -0.04344421259793468 -0.0315640680481058 rpy=-0.7989541677433551 -0.6090169187607924 -0.5313896516603533, axis 1 0 0
- added joint front_right_roller11_joint: type continuous, parent front_right_wheel_link, child front_right_roller11_link, origin xyz=0 -0.026850000000000023 -0.04650556418322434 rpy=-1.1831996401397156 -0.3613671239067081 -0.7137243789447655, axis 1 0 0
- added joint front_right_roller12_joint: type continuous, parent front_right_wheel_link, child front_right_roller12_link, origin xyz=0 -0.0056131784774729855 -0.05340582578127628 rpy=-1.4966127917301506 -0.07398025001120935 -0.7826515949744619, axis 1 0 0
- added joint front_right_roller13_joint: type continuous, parent front_right_wheel_link, child front_right_roller13_link, origin xyz=0 0.01659421259793466 -0.051071734925049746 rpy=1.3449626171032882 0.22028527385474703 -0.7603177925108144, axis 1 0 0
- added joint front_right_roller14_joint: type continuous, parent front_right_wheel_link, child front_right_roller14_link, origin xyz=0 0.03593231356147066 -0.039906877128136085 rpy=1.0038406803226874 0.4928592704898482 -0.6390993414905143, axis 1 0 0
- added joint front_right_roller15_joint: type continuous, parent front_right_wheel_link, child front_right_roller15_link, origin xyz=0 0.04905739107540767 -0.021841757733170465 rpy=0.5619350361043127 0.7022987807291682 -0.38630030387691144, axis 1 0 0
- added joint front_right_roller1_joint: type continuous, parent front_right_wheel_link, child front_right_roller1_link, origin xyz=0 0.0537 0.0 rpy=-0.0 0.7853981633974482 0.0, axis 1 0 0
- added joint front_right_roller2_joint: type continuous, parent front_right_wheel_link, child front_right_roller2_link, origin xyz=0 0.049057391075407665 0.02184175773317047 rpy=-0.5619350361043128 0.702298780729168 0.3863003038769115, axis 1 0 0
- added joint front_right_roller3_joint: type continuous, parent front_right_wheel_link, child front_right_roller3_link, origin xyz=0 0.03593231356147068 0.03990687712813607 rpy=-1.0038406803226867 0.4928592704898485 0.6390993414905141, axis 1 0 0
- added joint front_right_roller4_joint: type continuous, parent front_right_wheel_link, child front_right_roller4_link, origin xyz=0 0.016594212597934678 0.051071734925049746 rpy=-1.3449626171032882 0.2202852738547472 0.7603177925108144, axis 1 0 0
- added joint front_right_roller5_joint: type continuous, parent front_right_wheel_link, child front_right_roller5_link, origin xyz=0 -0.005613178477472996 0.05340582578127627 rpy=1.4966127917301504 -0.07398025001120949 0.7826515949744619, axis 1 0 0
- added joint front_right_roller6_joint: type continuous, parent front_right_wheel_link, child front_right_roller6_link, origin xyz=0 -0.026849999999999985 0.04650556418322435 rpy=1.1831996401397162 -0.3613671239067076 0.7137243789447657, axis 1 0 0
- added joint front_right_roller7_joint: type continuous, parent front_right_wheel_link, child front_right_roller7_link, origin xyz=0 -0.04344421259793467 0.03156406804810581 rpy=0.7989541677433554 -0.6090169187607923 0.5313896516603536, axis 1 0 0
- added joint front_right_roller8_joint: type continuous, parent front_right_wheel_link, child front_right_roller8_link, origin xyz=0 -0.05252652615940536 0.011164857796913676 rpy=0.2920075036845471 -0.7637777909460687 0.20499125187874387, axis 1 0 0
- added joint front_right_roller9_joint: type continuous, parent front_right_wheel_link, child front_right_roller9_link, origin xyz=0 -0.052526526159405354 -0.011164857796913686 rpy=-0.29200750368454736 -0.7637777909460687 -0.20499125187874406, axis 1 0 0
- added joint rear_left_roller10_joint: type continuous, parent rear_left_wheel_link, child rear_left_roller10_link, origin xyz=0 -0.04344421259793468 -0.0315640680481058 rpy=-0.7989541677433551 -0.6090169187607924 -0.5313896516603533, axis 1 0 0
- added joint rear_left_roller11_joint: type continuous, parent rear_left_wheel_link, child rear_left_roller11_link, origin xyz=0 -0.026850000000000023 -0.04650556418322434 rpy=-1.1831996401397156 -0.3613671239067081 -0.7137243789447655, axis 1 0 0
- added joint rear_left_roller12_joint: type continuous, parent rear_left_wheel_link, child rear_left_roller12_link, origin xyz=0 -0.0056131784774729855 -0.05340582578127628 rpy=-1.4966127917301506 -0.07398025001120935 -0.7826515949744619, axis 1 0 0
- added joint rear_left_roller13_joint: type continuous, parent rear_left_wheel_link, child rear_left_roller13_link, origin xyz=0 0.01659421259793466 -0.051071734925049746 rpy=1.3449626171032882 0.22028527385474703 -0.7603177925108144, axis 1 0 0
- added joint rear_left_roller14_joint: type continuous, parent rear_left_wheel_link, child rear_left_roller14_link, origin xyz=0 0.03593231356147066 -0.039906877128136085 rpy=1.0038406803226874 0.4928592704898482 -0.6390993414905143, axis 1 0 0
- added joint rear_left_roller15_joint: type continuous, parent rear_left_wheel_link, child rear_left_roller15_link, origin xyz=0 0.04905739107540767 -0.021841757733170465 rpy=0.5619350361043127 0.7022987807291682 -0.38630030387691144, axis 1 0 0
- added joint rear_left_roller1_joint: type continuous, parent rear_left_wheel_link, child rear_left_roller1_link, origin xyz=0 0.0537 0.0 rpy=-0.0 0.7853981633974482 0.0, axis 1 0 0
- added joint rear_left_roller2_joint: type continuous, parent rear_left_wheel_link, child rear_left_roller2_link, origin xyz=0 0.049057391075407665 0.02184175773317047 rpy=-0.5619350361043128 0.702298780729168 0.3863003038769115, axis 1 0 0
- added joint rear_left_roller3_joint: type continuous, parent rear_left_wheel_link, child rear_left_roller3_link, origin xyz=0 0.03593231356147068 0.03990687712813607 rpy=-1.0038406803226867 0.4928592704898485 0.6390993414905141, axis 1 0 0
- added joint rear_left_roller4_joint: type continuous, parent rear_left_wheel_link, child rear_left_roller4_link, origin xyz=0 0.016594212597934678 0.051071734925049746 rpy=-1.3449626171032882 0.2202852738547472 0.7603177925108144, axis 1 0 0
- added joint rear_left_roller5_joint: type continuous, parent rear_left_wheel_link, child rear_left_roller5_link, origin xyz=0 -0.005613178477472996 0.05340582578127627 rpy=1.4966127917301504 -0.07398025001120949 0.7826515949744619, axis 1 0 0
- added joint rear_left_roller6_joint: type continuous, parent rear_left_wheel_link, child rear_left_roller6_link, origin xyz=0 -0.026849999999999985 0.04650556418322435 rpy=1.1831996401397162 -0.3613671239067076 0.7137243789447657, axis 1 0 0
- added joint rear_left_roller7_joint: type continuous, parent rear_left_wheel_link, child rear_left_roller7_link, origin xyz=0 -0.04344421259793467 0.03156406804810581 rpy=0.7989541677433554 -0.6090169187607923 0.5313896516603536, axis 1 0 0
- added joint rear_left_roller8_joint: type continuous, parent rear_left_wheel_link, child rear_left_roller8_link, origin xyz=0 -0.05252652615940536 0.011164857796913676 rpy=0.2920075036845471 -0.7637777909460687 0.20499125187874387, axis 1 0 0
- added joint rear_left_roller9_joint: type continuous, parent rear_left_wheel_link, child rear_left_roller9_link, origin xyz=0 -0.052526526159405354 -0.011164857796913686 rpy=-0.29200750368454736 -0.7637777909460687 -0.20499125187874406, axis 1 0 0
- added joint rear_right_roller10_joint: type continuous, parent rear_right_wheel_link, child rear_right_roller10_link, origin xyz=0 -0.04344421259793468 -0.0315640680481058 rpy=-0.7989541677433551 0.6090169187607924 0.5313896516603533, axis 1 0 0
- added joint rear_right_roller11_joint: type continuous, parent rear_right_wheel_link, child rear_right_roller11_link, origin xyz=0 -0.026850000000000023 -0.04650556418322434 rpy=-1.1831996401397156 0.3613671239067081 0.7137243789447655, axis 1 0 0
- added joint rear_right_roller12_joint: type continuous, parent rear_right_wheel_link, child rear_right_roller12_link, origin xyz=0 -0.0056131784774729855 -0.05340582578127628 rpy=-1.4966127917301506 0.07398025001120935 0.7826515949744619, axis 1 0 0
- added joint rear_right_roller13_joint: type continuous, parent rear_right_wheel_link, child rear_right_roller13_link, origin xyz=0 0.01659421259793466 -0.051071734925049746 rpy=1.3449626171032882 -0.22028527385474703 0.7603177925108144, axis 1 0 0
- added joint rear_right_roller14_joint: type continuous, parent rear_right_wheel_link, child rear_right_roller14_link, origin xyz=0 0.03593231356147066 -0.039906877128136085 rpy=1.0038406803226874 -0.4928592704898482 0.6390993414905143, axis 1 0 0
- added joint rear_right_roller15_joint: type continuous, parent rear_right_wheel_link, child rear_right_roller15_link, origin xyz=0 0.04905739107540767 -0.021841757733170465 rpy=0.5619350361043127 -0.7022987807291682 0.38630030387691144, axis 1 0 0
- added joint rear_right_roller1_joint: type continuous, parent rear_right_wheel_link, child rear_right_roller1_link, origin xyz=0 0.0537 0.0 rpy=-0.0 -0.7853981633974482 -0.0, axis 1 0 0
- added joint rear_right_roller2_joint: type continuous, parent rear_right_wheel_link, child rear_right_roller2_link, origin xyz=0 0.049057391075407665 0.02184175773317047 rpy=-0.5619350361043128 -0.702298780729168 -0.3863003038769115, axis 1 0 0
- added joint rear_right_roller3_joint: type continuous, parent rear_right_wheel_link, child rear_right_roller3_link, origin xyz=0 0.03593231356147068 0.03990687712813607 rpy=-1.0038406803226867 -0.4928592704898485 -0.6390993414905141, axis 1 0 0
- added joint rear_right_roller4_joint: type continuous, parent rear_right_wheel_link, child rear_right_roller4_link, origin xyz=0 0.016594212597934678 0.051071734925049746 rpy=-1.3449626171032882 -0.2202852738547472 -0.7603177925108144, axis 1 0 0
- added joint rear_right_roller5_joint: type continuous, parent rear_right_wheel_link, child rear_right_roller5_link, origin xyz=0 -0.005613178477472996 0.05340582578127627 rpy=1.4966127917301504 0.07398025001120949 -0.7826515949744619, axis 1 0 0
- added joint rear_right_roller6_joint: type continuous, parent rear_right_wheel_link, child rear_right_roller6_link, origin xyz=0 -0.026849999999999985 0.04650556418322435 rpy=1.1831996401397162 0.3613671239067076 -0.7137243789447657, axis 1 0 0
- added joint rear_right_roller7_joint: type continuous, parent rear_right_wheel_link, child rear_right_roller7_link, origin xyz=0 -0.04344421259793467 0.03156406804810581 rpy=0.7989541677433554 0.6090169187607923 -0.5313896516603536, axis 1 0 0
- added joint rear_right_roller8_joint: type continuous, parent rear_right_wheel_link, child rear_right_roller8_link, origin xyz=0 -0.05252652615940536 0.011164857796913676 rpy=0.2920075036845471 0.7637777909460687 -0.20499125187874387, axis 1 0 0
- added joint rear_right_roller9_joint: type continuous, parent rear_right_wheel_link, child rear_right_roller9_link, origin xyz=0 -0.052526526159405354 -0.011164857796913686 rpy=-0.29200750368454736 0.7637777909460687 0.20499125187874406, axis 1 0 0
- joint front_left_wheel_joint: axis 0 1.0 0 -> 1 0 0; origin xyz=0.1 0.1 0.01535 rpy=0 0 0 -> xyz=0.1 0.1 0.01535 rpy=0 0 1.5707963267948966
- joint front_right_wheel_joint: axis 0 1.0 0 -> 1 0 0; origin xyz=0.1 -0.1 0.01535 rpy=0 0 0 -> xyz=0.1 -0.1 0.01535 rpy=0 0 1.5707963267948966
- joint rear_left_wheel_joint: axis 0 1.0 0 -> 1 0 0; origin xyz=-0.1 0.1 0.01535 rpy=0 0 0 -> xyz=-0.1 0.1 0.01535 rpy=0 0 1.5707963267948966
- joint rear_right_wheel_joint: axis 0 1.0 0 -> 1 0 0; origin xyz=-0.1 -0.1 0.01535 rpy=0 0 0 -> xyz=-0.1 -0.1 0.01535 rpy=0 0 1.5707963267948966
