Commit message: 2024.04.17 dea, stl文件重新上传；任务目标修正为将A球拉至0点位置

File: assets/urdf/robomasterEP_description/robot/robomaster.urdf (robot description, URDF)
Before this commit: robot robomaster_ep, 99 links, 98 joints
Joints:
- joint front_left_wheel_joint: limit effort=30 velocity=1.0 -> effort=30 velocity=5
- joint front_right_wheel_joint: limit effort=30 velocity=1.0 -> effort=30 velocity=5
- joint rear_left_wheel_joint: limit effort=30 velocity=1.0 -> effort=30 velocity=5
- joint rear_right_wheel_joint: limit effort=30 velocity=1.0 -> effort=30 velocity=5

Commit message: 2024.04.19麦轮运动学速度控制，并删除了关节limit

File: assets/urdf/robomasterEP_description/robot/robomaster.urdf (robot description, URDF)
Before this commit: robot robomaster_ep, 99 links, 98 joints
Joints:
- joint front_left_wheel_joint: limit effort=30 velocity=5 -> (none)
- joint front_right_wheel_joint: limit effort=30 velocity=5 -> (none)
- joint rear_left_wheel_joint: limit effort=30 velocity=5 -> (none)
- joint rear_right_wheel_joint: limit effort=30 velocity=5 -> (none)

Commit message: 2024.04.28添加了apollo任务（包括两个apollo与一个obstacle），将rm的钳子改为位置控制，未添加力传感，有碰撞时仍无法正确搜寻目标

File: assets/urdf/robomasterEP_description/robot/robomaster.urdf (robot description, URDF)
Before this commit: robot robomaster_ep, 99 links, 98 joints
Links:
- link chassis_base_link: mass 9.934 -> 100

Commit message: 2024.05.10rm有碰撞找球成功，添加darwin机器人但其关节还受到未知力的影响

File: assets/urdf/robomasterEP_description/robot/robomaster.urdf (robot description, URDF)
Before this commit: robot robomaster_ep, 99 links, 98 joints
Joints:
- joint left_gripper_joint_1: limit lower=-0.4 upper=0 effort=10 velocity=5 -> lower=-0.4 upper=0 effort=20 velocity=20
- joint right_gripper_joint_1: limit lower=0 upper=0.4 effort=10 velocity=5 -> lower=0 upper=0.4 effort=20 velocity=20

Commit message: 2024.05.16添加足球模型，可有碰撞找球，改善darwin自碰撞

File: assets/urdf/robomasterEP_description/robot/robomaster.urdf (robot description, URDF)
Before this commit: robot robomaster_ep, 99 links, 98 joints
Joints:
- joint left_gripper_joint_1: limit lower=-0.4 upper=0 effort=20 velocity=20 -> lower=-0.4 upper=0 effort=1 velocity=20
- joint right_gripper_joint_1: limit lower=0 upper=0.4 effort=20 velocity=20 -> lower=0 upper=0.4 effort=1 velocity=20
