Commit message: 2024.05.29添加了robomasterfull

File: assets/urdf/robomasterEP_description/robot/robomaster_full.urdf (robot description, URDF)
Before this commit: robot robomaster_ep, 99 links, 98 joints
Joints:
- joint arm_1_joint: origin xyz=0.0103961 -0.0255713 0.030741 rpy=0 1.3 0 -> xyz=0.0103961 -0.0255713 0.030741 rpy=0 0 0; type fixed -> revolute
- joint arm_2_joint: origin xyz=0.0018704 0.0438659 0.1210238 rpy=0 -0.5 0 -> xyz=0.0018704 0.0438659 0.1210238 rpy=0 0 0; type fixed -> revolute
- joint endpoint_bracket_joint: type fixed -> revolute
- joint gripper_joint: origin xyz=0.0002793 -0.027026 0.0001815 rpy=0 -0.8 0 -> xyz=0.0002793 -0.027026 0.0001815 rpy=0 0 0
- joint left_gripper_joint_2: type fixed -> revolute
- joint left_gripper_joint_5: type fixed -> revolute
- joint right_gripper_joint_2: type fixed -> revolute
- joint right_gripper_joint_5: type fixed -> revolute
- joint rod_2_joint: origin xyz=-0.0224276 -0.0290701 0.0554782 rpy=0 1.3 0 -> xyz=-0.0224276 -0.0290701 0.0554782 rpy=0 0 0
- joint rod_3_joint: origin xyz=-0.042397 0.0004533 0.0223131 rpy=0 0.5 0 -> xyz=-0.042397 0.0004533 0.0223131 rpy=0 0 0
- joint rod_joint: origin xyz=0.009805 0.0214241 0.0319234 rpy=0 0.8 0 -> xyz=0.009805 0.0214241 0.0319234 rpy=0 0 0
- joint triangle_joint: origin xyz=0.0020224 -0.007103 0.1212334 rpy=0 -1.1 0 -> xyz=0.0020224 -0.007103 0.1212334 rpy=0 0 0

Commit message: 2024.06.05添加了robomaster的具身控制，可以控制钳子去找球

File: assets/urdf/robomasterEP_description/robot/robomaster_full.urdf (robot description, URDF)
Before this commit: robot robomaster_ep, 99 links, 98 joints
Links:
- removed link rod_1_link
- removed link rod_2_link
- removed link rod_3_link
- removed link rod_link
- removed link triangle_link
Joints:
- removed joint rod_1_joint
- removed joint rod_2_joint
- removed joint rod_3_joint
- removed joint rod_joint
- removed joint triangle_joint
- joint arm_1_joint: limit lower=-0.274 upper=1.384 effort=1 velocity=1 -> (none)
- joint arm_2_joint: limit effort=1 velocity=1 -> (none); mimic joint=rod_3_joint multiplier=-1.0 offset=0.0 -> (none)
- joint endpoint_bracket_joint: mimic joint=rod_joint multiplier=-1.0 offset=0.0 -> (none)
- joint left_gripper_joint_1: limit lower=-0.4 upper=0 effort=1 velocity=20 -> lower=-0.4 upper=0
- joint left_gripper_joint_2: type revolute -> fixed
- joint left_gripper_joint_5: type revolute -> fixed
- joint right_gripper_joint_1: limit lower=0 upper=0.4 effort=1 velocity=20 -> lower=0 upper=0.4
- joint right_gripper_joint_2: type revolute -> fixed
- joint right_gripper_joint_5: type revolute -> fixed
